Commit message: Add lidar in go2

File: robots/go2_description/xacro/gazebo.xacro (robot description, xacro)
@@ -54,4 +54,55 @@
         </sensor>
     </gazebo>
+    <gazebo reference="lidar_link">
+        <sensor name="lidar_sensor" type="ray">
+            <always_on>true</always_on>
+            <pose>0 0 0 1.570796 -0.32 0</pose>
+            <!-- <pose>0 0 0 0 0 0</pose> -->
+            <visualize>false</visualize>
+            <update_rate>30</update_rate>
+            <ray>
+                <scan>
+                    <horizontal>
+                        <samples>1024</samples>
+                        <resolution>1</resolution>
+                        <min_angle>-3.14159265359</min_angle>
+                        <max_angle>3.14159265359</max_angle>
+                    </horizontal>
+                    <vertical>
+                        <samples>16</samples>
+                        <resolution>1</resolution>
+                        <min_angle>-0.785398</min_angle>
+                        <max_angle>0.785398</max_angle>
+                    </vertical>
+                    <!-- <horizontal>
+                        <samples>1024</samples>
+                        <resolution>1</resolution>
+                        <min_angle>-3.14159265359</min_angle>
+                        <max_angle>3.14159265359</max_angle>
+                    </horizontal>
+                    <vertical>
+                        <samples>16</samples>
+                        <resolution>1</resolution>
+                        <min_angle>-0.261799387799</min_angle>
+                        <max_angle> 0.261799387799</max_angle>
+                    </vertical> -->
+                </scan>
+                <range>
+                    <min>0.05</min>
+                    <max>30.0</max>
+                    <resolution>0.001</resolution>
+                </range>
+                <noise>
+                    <type>gaussian</type>
+                    <mean>0.0</mean>
+                    <stddev>0.00</stddev>
+                </noise>
+            </ray>
+            <plugin name="gazebo_ros_laser" filename="libgazebo_ros_velodyne_laser.so">
+                <topicName>/go2_gazebo/velodyne_points</topicName>
+                <frameName>lidar_link</frameName>
+            </plugin>
+        </sensor>
+    </gazebo>
     <!-- Foot contacts. -->
     <gazebo reference="FR_calf">

File: robots/go2_description/xacro/robot.xacro (robot description, xacro)
@@ -81,4 +81,29 @@
         </collision>
     </link>
+    <joint name="lidar_joint" type="fixed">
+        <parent link="trunk"/>
+        <child link="lidar_link"/>
+        <origin rpy="0 -0.32 0" xyz="0.275 0 -0.04"/>
+    </joint>
+    <link name="lidar_link">
+        <inertial>
+            <mass value="0.001"/>
+            <origin rpy="0 0 0" xyz="0 0 0"/>
+            <inertia ixx="0.0001" ixy="0" ixz="0" iyy="0.0001" iyz="0" izz="0.0001"/>
+        </inertial>
+        <visual>
+            <origin rpy="0 0 0" xyz="0 0 0"/>
+            <geometry>
+                <box size="0.001 0.001 0.001"/>
+            </geometry>
+            <!-- <material name="red"/> -->
+        </visual>
+        <collision>
+            <origin rpy="0 0 0" xyz="0 0 0"/>
+            <geometry>
+                <box size=".001 .001 .001"/>
+            </geometry>
+        </collision>
+    </link>
     <!--
     <joint name="load_joint" type="fixed">
@@ -106,5 +131,5 @@
         </collision>
     </link>
--->
+    -->
     <xacro:leg name="FR" mirror="-1" mirror_dae= "False" front_hind="1"  front_hind_dae="True"  />
     <xacro:leg name="FL" mirror="1"  mirror_dae="True"   front_hind="1"  front_hind_dae="True"  />
